File: 1130MRAM.kicad_pcb (KiCad board)
At the start: 4 copper layers, 228.6 x 63.5 mm, 152 parts, among them IC1 BSV52LT1G, IC10 BSV52LT1G, IC11 BSV52LT1G, IC12 BSV52LT1G, IC13 BSV52LT1G, IC14 BSV52LT1G, IC15 BSV52LT1G, IC16 BSV52LT1G, IC17 BSV52LT1G, IC18 BSV52LT1G, IC2 BSV52LT1G, IC3 BSV52LT1G, IC4 BSV52LT1G, IC5 BSV52LT1G, IC6 BSV52LT1G, IC7 BSV52LT1G, IC8 BSV52LT1G, IC9 BSV52LT1G, J1 Conn_01x09_MountingPin, J1A09 SLTpad, J1A11 SLTpad, J2 Conn_01x09_MountingPin, J3 Conn_01x09_MountingPin, J4 Conn_01x09_MountingPin, J5 Screw_Terminal_01x03, K1E09 SLTpad, K1E11 SLTpad, M1A09 SLTpad, M1A11 SLTpad, M1C09 SLTpad, M1D09 SLTpad, M1E09 SLTpad, M1E11 SLTpad, SW1 SLTpad, U1 MR0A16AYS35, U10 74LVC08A, U11 74LVC08A, U14 74HC00, U15 74HC86, U16 74HC86, U17 74HC86, U18 74HC86, U2 SN74LV240APWR, U3 SN74LV240APWR, U4 LDL1117, U5 LDL1117, U6 74LVC1G14, U7 74LVC08A, U8 74LVC08A, U9 74LVC08A

Commit message: Final version of the board and bill of material
Parts:
- added J6: Screw_Terminal_01x01, TerminalBlock_WAGO:TerminalBlock_WAGO_236-101_1x01_P5.00mm_45Degree, F.Cu at (252.1, 111.3)
- J5: footprint Connector_Phoenix_MC_HighVoltage:PhoenixContact_MCV_1,5_2-G-5.08_1x02_P5.08mm_Vertical -> TerminalBlock_WAGO:TerminalBlock_WAGO_236-102_1x02_P5.00mm_45Degree
- R11, R14, R15, R16, R17, R18, R19, R20, R21, R22, R23, R24, R3, R4, R5, R6: value 2k -> 470
- R12, R13: value 2K -> 470
- moved J5 0.75 mm to (110.5, 101.3)
Routing:
- net +3.3V: track 401.1 -> 411.3 mm, vias 103 -> 107
- net Net-(R21-Pad2): track 84.7 -> 86.3 mm
Other:
- board text added: "Braided Ground"

Commit message: Improved PCB design
improved ground paths for MRAM chiip, added 10uF decoupling capacitor next to .1uF capacitor. 

opened solder mask for four ground pads to solder magnetic shield over chip
Parts:
- added C6: 10uF, Capacitor_SMD:C_0805_2012Metric, B.Cu at (148.9, 97.5)
Routing:
- net GND: track 262.5 -> 269.7 mm, vias 87 -> 89
- net +3.3V: track 411.3 -> 413.7 mm
Other:
- board text added: "+"
